File: IEMU_Base_DB/feedback+interaction.kicad_sch (KiCad schematic)
At the start: 35 parts, among them J401 SJ3-35083C-TR, Q401 CSD13381F4, SW401 TS-1088-AR02016, U401 SN74LVC1T45DCKR

Commit message: added hall effect sensor for lid detection
Parts:
- added C403: 100n, Capacitor_SMD:C_0402_1005Metric, symbol 0_Passives:C_100nF_0402
- added U402: DRV5032FADBZR, Package_TO_SOT_SMD:SOT-23, symbol 0_Sensors:DRV5032FADBZ
Connections:
- net +1V8_MCU: now also C403.1, U402.1 (VCC)
- net GND: now also C403.2, U402.3 (GND)
- new net LID_SENSE: U402.2 (OUT)
Other:
- note added: "Connector, Lid-Sensor, LEDs & Buttons"
- note added: "Lid-Hall-Effect-Sensor"
- note removed: "Connector, LEDs & Buttons"
- moved on the sheet: MH401, MH402, MH403, MH404, SW401, TP404
