File: IEMU_Base_DB/feedback+interaction.kicad_sch (KiCad schematic)
At the start: 38 parts, among them J401 SJ3-35083C-TR, Q401 CSD13381F4, SW401 TS-1088-AR02016, U401 SN74LVC1T45DCKR, U402 DRV5032FADBZR

Commit message: added header pins
Parts:
- MH401, MH402, MH403, MH404: footprint (none) -> MountingHole:MountingHole_2.2mm_M2_Pad_Via
Changed lines of the file:
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@@
 			)
 		)
-		(property "Footprint" ""
+		(property "Footprint" "MountingHole:MountingHole_2.2mm_M2_Pad_Via"
 			(at 119.38 170.18 0)
 			(effects
@@
 			)
 		)
-		(property "Footprint" ""
+		(property "Footprint" "MountingHole:MountingHole_2.2mm_M2_Pad_Via"
 			(at 127 170.18 0)
 			(effects
@@
 			)
 		)
-		(property "Footprint" ""
+		(property "Footprint" "MountingHole:MountingHole_2.2mm_M2_Pad_Via"
 			(at 111.76 170.18 0)
 			(effects
@@
 			)
 		)
-		(property "Footprint" ""
+		(property "Footprint" "MountingHole:MountingHole_2.2mm_M2_Pad_Via"
 			(at 134.62 170.18 0)
 			(effects
