File: IEMU_Base_DB/mcu+peripherals.kicad_sch (KiCad schematic)
At the start: 27 parts, among them J301 Conn_ARM_SWD_TagConnect_TC203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, J302 503398-1892, U301 Ezurio BL54L15, U302 TMUX1204DQAR, Y201 32.768kHz

Commit message: added hall effect sensor for lid detection
Connections:
- net LID_SENSE: now reaches U301.3 (P2.08)
- no-connect marks 3 -> 2
Changed lines of the file:
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@@
-	)
-	(no_connect
-		(at 48.26 97.79)
 	)
 	(no_connect
@@
 		(pts
 			(xy 194.31 48.26) (xy 194.31 55.88)
+		)
+		(stroke
+			(width 0)
+			(type default)
+		)
+	)
+	(wire
+		(pts
+			(xy 39.37 97.79) (xy 48.26 97.79)
 		)
 		(stroke
@@
 		)
 	)
+	(hierarchical_label "LID_SENSE"
+		(shape output)
+		(at 39.37 97.79 180)
+		(effects
+			(font
+				(size 1.27 1.27)
+			)
+			(justify right)
+		)
+	)
