File: IEMU_Base_DB/IEMU_Base_DB.kicad_pcb (KiCad board)
At the start: 4 copper layers, 169 parts, among them J101 USB4125-GF-A, J102 Conn_01x02_Pin, J201 DF13-4P-1.25H(21), J202 DF13-4P-1.25H(21), J203 DF13-4P-1.25H(21), J204 DF13-4P-1.25H(21), J301 Conn_ARM_SWD_TagConnect_TC203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, J302 503398-1892, J401 SJ3-35083C-TR, Q101 CSD85301Q2, Q401 CSD13381F4, SW401 TS-1088-AR02016, U101 NPM1300-QEAA-R7, U102 BQ29702DSER, U103 TPS61099DRV, U104 INA216A2RSWR, U201 TPS2553DRVT, U202 TPS2553DRVT, U203 TPS2553DRVT, U204 TPS2553DRVT, U301 Ezurio BL54L15, U302 TMUX1204DQAR, U401 SN74LVC1T45DCKR, U402 DRV5032FADBZR, Y201 32.768kHz

Commit message: added header pins
Parts:
- added J103: ~, 0_Connectors:SAMTEC_MTSW-101-X-X-D-X, F.Cu at (222.0, 112.2)
- added J104: ~, 0_Connectors:SAMTEC_MTSW-101-X-X-D-X, F.Cu at (213.0, 113.5)
- added J105: ~, 0_Connectors:SAMTEC_MTSW-101-X-X-D-X, F.Cu at (221.2, 102.9)
- added MH401: MountingHole_Pad, MountingHole:MountingHole_2.2mm_M2_Pad_Via, F.Cu at (246.5, 138.8)
- added MH402: MountingHole_Pad, MountingHole:MountingHole_2.2mm_M2_Pad_Via, F.Cu at (246.5, 82.8)
- added MH403: MountingHole_Pad, MountingHole:MountingHole_2.2mm_M2_Pad_Via, F.Cu at (192.5, 87.2)
- added MH404: MountingHole_Pad, MountingHole:MountingHole_2.2mm_M2_Pad_Via, F.Cu at (192.5, 138.8)
- moved R101 87.7 mm to (215.0, 125.0), turned to 180 degrees
- moved R102 85.8 mm to (215.0, 124.0), turned to 180 degrees
- moved C106 85.3 mm to (221.2, 117.5)
- moved C302 83.6 mm to (228.5, 93.5), turned to -90 degrees
- moved C112 83.2 mm to (224.2, 117.8), turned to -90 degrees
- moved C107 81.4 mm to (218.2, 117.5), turned to 180 degrees
- moved R110 80.1 mm to (223.2, 108.2), turned to 90 degrees
- moved U302 79.6 mm to (227.0, 106.3), turned to 90 degrees
- moved L102 76.5 mm to (222.0, 116.0), turned to 180 degrees
- moved C109 75.5 mm to (217.6, 112.0)
- moved L103 74.9 mm to (218.2, 115.0), turned to -90 degrees
- moved C113 74.0 mm to (216.8, 115.0), turned to -90 degrees
- moved L101 71.2 mm to (217.6, 110.5)
- moved D305 71.1 mm to (232.8, 86.2), turned to -90 degrees
- moved D304 70.9 mm to (232.8, 84.4), turned to 90 degrees
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Connections:
- net /3_nRF Module & SDCard/SDIO_CLK_SD renamed /3_nRF Module & SDCard/SPI_SD_CLK_CONN
- net /3_nRF Module & SDCard/SDIO_CMD_SD renamed /3_nRF Module & SDCard/SPI_SD_MOSI_CONN
- net /3_nRF Module & SDCard/SDIO_D3_SD renamed /3_nRF Module & SDCard/SPI_SD_CS_CONN
- net Net-(U101-VSET2) renamed /1_Power/NPM_VSET2
- C110 pad 1: +5V0 -> Net-(U103-VOUT)
- C111 pad 1: +5V0 -> Net-(U103-VOUT)
- C113 pad 1: +3V0 -> /1_Power/NPM_VOUT2
- FL301 pad 10: /3_nRF Module & SDCard/SDIO_D0_SD -> /3_nRF Module & SDCard/SPI_SD_MISO_MCU
- FL301 pad 14: /3_nRF Module & SDCard/SDIO_D2_SD -> /3_nRF Module & SDCard/SPI_SD_D2_CONN
- FL301 pad 9: /3_nRF Module & SDCard/SDIO_D1_SD -> /3_nRF Module & SDCard/SPI_SD_D2_CONN
- J302 pad 1: /3_nRF Module & SDCard/SDIO_D2_SD -> /3_nRF Module & SDCard/SPI_SD_D2_CONN
- J302 pad 7: /3_nRF Module & SDCard/SDIO_D0_SD -> /3_nRF Module & SDCard/SPI_SD_MISO_MCU
- J302 pad 8: /3_nRF Module & SDCard/SDIO_D1_SD -> /3_nRF Module & SDCard/SPI_SD_D2_CONN
- L103 pad 1: +3V0 -> /1_Power/NPM_VOUT2
- R108 pad 2: +5V0 -> Net-(U103-VOUT)
- R110 pad 1: /1_Power/NPM_VOUT1 -> /1_Power/Header_Shunt_CM
- TP107 pad 1: +5V0 -> Net-(U103-VOUT)
- TP306 pad 1: /3_nRF Module & SDCard/SDIO_D0_SD -> /3_nRF Module & SDCard/SPI_SD_MISO_MCU
- U101 pad 32: +3V0 -> /1_Power/NPM_VOUT2
- U103 pad 2: +5V0 -> Net-(U103-VOUT)
- U104 pad 2: /1_Power/NPM_VOUT1 -> /1_Power/Header_Shunt_CM
- U104 pad 3: /1_Power/NPM_VOUT1 -> /1_Power/Header_Shunt_CM
Routing:
- net /1_Power/NPM_VOUT2: track 0.00 -> 9.74 mm, vias 0 -> 2
- added copper zone on F.Cu, net +3V0
Other:
- board outline added: 60 x 62 mm
