File: IEMU_Base_DB/mcu+sd.kicad_sch (KiCad schematic)
At the start: 27 parts, among them J301 Conn_ARM_SWD_TagConnect_TC203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, J302 503398-1892, U301 Ezurio BL54L15, U302 TMUX1204DQAR, Y201 32.768kHz

Commit message: added header pins
Connections:
- net SDIO_D0_SD is gone; now on net SPI_SD_MISO_MCU: FL301.10 (DAT0_EX), J302.7 (DAT0), TP306.1
- net SDIO_D2_SD is gone; now on net SPI_SD_D2_CONN: FL301.14 (DAT2_EX), J302.1 (DAT2)
- net SDIO_CLK_SD renamed SPI_SD_CLK_CONN
- net SDIO_CMD_SD renamed SPI_SD_MOSI_CONN
- net SDIO_D1_SD renamed SPI_SD_D2_CONN
- net SDIO_D3_SD renamed SPI_SD_CS_CONN
Changed lines of the file:
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@@
 		)
 	)
-	(label "SDIO_D0_SD"
+	(label "SPI_SD_MISO_MCU"
 		(at 222.25 110.49 0)
 		(effects
@@
 		)
 	)
-	(label "SDIO_D1_SD"
+	(label "SPI_SD_D2_CONN"
 		(at 222.25 113.03 0)
 		(effects
@@
 		)
 	)
-	(label "SDIO_D2_SD"
+	(label "SPI_SD_D2_CONN"
 		(at 222.25 100.33 0)
 		(effects
@@
 		)
 	)
-	(label "SDIO_D3_SD"
+	(label "SPI_SD_CS_CONN"
 		(at 222.25 102.87 0)
 		(effects
@@
 		)
 	)
-	(label "SDIO_CLK_SD"
+	(label "SPI_SD_CLK_CONN"
 		(at 222.25 107.95 0)
 		(effects
@@
 		)
 	)
-	(label "SDIO_CMD_SD"
+	(label "SPI_SD_MOSI_CONN"
 		(at 222.25 105.41 0)
 		(effects
