File: IEMU_Base_DB/power.kicad_sch (KiCad schematic)
At the start: 51 parts, among them J101 USB4125-GF-A, J102 Conn_01x02_Pin, Q101 CSD85301Q2, U101 NPM1300-QEAA-R7, U102 BQ29702DSER, U103 TPS61099DRV, U104 INA216A2RSWR

Commit message: added header pins
Parts:
- added J103, J104, J105: ~, 0_Connectors:SAMTEC_MTSW-101-X-X-D-X, symbol 0_Connectors:MTSW-101-X-X-D-X
Connections:
- net +3V0: now also J104.02; no longer C113.1, L103.1, U101.32 (VOUT2)
- net +5V0: now also J105.02; no longer C110.1, C111.1, R108.2, TP107.1, U103.2 (VOUT)
- net NPM_VOUT1: now also J103.01; no longer R110.1, U104.2 (IN+), U104.3 (IN+)
- net NPM_VSET2: now reaches R102.1, U101.16 (VSET2)
- new net: C110.1, C111.1, J105.01, R108.2, TP107.1, U103.2 (VOUT)
- new net Header_Shunt_CM: J103.02, R110.1, U104.2 (IN+), U104.3 (IN+)
- new net NPM_VOUT2: C113.1, J104.01, L103.1, U101.32 (VOUT2)
Other:
- moved on the sheet: R110, TP105, TP109, U104
