File: IEMU_Sensor_DB/power.kicad_sch (KiCad schematic)
At the start: 60 parts, among them J101 USB4125-GF-A, J102 DF13-4P-1.25H(21), Q101 CSD85301Q2, U101 NPM1304-QEAA-R7, U102 BQ29702DSER, U103 TLV75530PDRVR, U104 INA216A2RSWR

Commit message: added header pins
Parts:
- added J103, J104, J105: ~, 0_Connectors:SAMTEC_MTSW-101-X-X-D-X, symbol 0_Connectors:MTSW-101-X-X-D-X
Connections:
- net +1V8_Peripherals: now also J104.02; no longer C112.1, L102.1, U101.32 (VOUT2)
- net +3V0: now also J105.02; no longer C110.1, TP105.1, U103.1 (OUT)
- net NPM_VOUT1: now also J103.01; no longer R108.1, U104.2 (IN+), U104.3 (IN+)
- new net: C112.1, J104.01, L102.1, U101.32 (VOUT2)
- new net: J103.02, R108.1, U104.2 (IN+), U104.3 (IN+)
- new net: C110.1, J105.01, TP105.1, U103.1 (OUT)

Commit message: commit after component purchase
Parts:
- removed D104, D105: PMEG3010ESBYL, 0_Power:DIODFN100X60X30-2N, symbol 0_Power:D_Schottky_PMEG3010ESBYL
- removed D107, D108: ESD9L1P8, Diode_SMD:D_SOD-882, symbol 0_Power:ESD9L1P8
- added D104, D105: CTS05S30, Diode_SMD:D_SOD-882, symbol 0_Power:D_Schottky_CTS05S30
- added D107, D108: RCLAMP01811PW.C, 0_Power:DIODFN100X60X55-2N, symbol 0_Power:RCLAMP01811PW.C
- R104: value 330 -> 330R
Connections:
- net +VBUS_IN: now also D104.2 (A), D105.2 (A)
- net +VBUS_IN_CONN: now also D105.1 (K)
- net +VBUS_IN_USB: now also D104.1 (K)
- net CHG_DOCK_DET_CONN: now also D108.1 (I/O)
- net CHG_DOCK_UART_CONN: now also D107.1 (I/O)
- net GND: now also D107.2 (GND), D108.2 (GND)
- net NPM_VOUT2: now reaches C112.1, J104.01, L102.1, U101.32 (VOUT2)
- net Shunt_CM_Header: now reaches J103.02, R108.1, U104.2 (IN+), U104.3 (IN+)
- net LDO_OUT: now reaches C110.1, J105.01, TP105.1, U103.1 (OUT)
- net NC: no longer names the net of U102.1 (NC)
- no-connect marks 7 -> 8
Other:
- note added: "Schottkey Diodes to prevent leakage of 5v into connector that is unused. 5V - 0.36V -> 4.64V still enough for PMIC"
- note removed: "Schottkey Diodes to prevent leakage of 5v into connector that is unused. 5V - 0.365V -> 4.635V still enough for PMIC"
