File: IEMU_Sensor_DB/IEMU_Sensor_DB.kicad_pcb (KiCad board)
At the start: 4 copper layers, 55 x 53 mm, 122 parts, among them J101 USB4125-GF-A, J102 DF13-4P-1.25H(21), J201 Conn_ARM_SWD_TagConnect_TC203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, J301 Conn_01x02_Pin, M401 VZ43FM1B8230001L, Q101 CSD85301Q2, Q301 CSD13381F4, Q302 CSD13381F4, Q303 CSD13381F4, Q304 CSD13381F4, SW301 NANOT_160_BP, SW302 TS-1088-AR02016, U101 NPM1304-QEAA-R7, U102 BQ29702DSER, U103 TLV75530PDRVR, U104 INA216A2RSWR, U201 Ezurio BL54L15, U202 W25N02JWZEIF, U203 LSM6DSV320XTR, U204 MMC5603NJ, Y201 32.768kHz

Commit message: commit after component purchase
Parts:
- added J103: ~, 0_Connectors:SAMTEC_MTSW-101-X-X-D-X, F.Cu at (119.0, 88.5)
- added J104: ~, 0_Connectors:SAMTEC_MTSW-101-X-X-D-X, F.Cu at (112.5, 96.0)
- added J105: ~, 0_Connectors:SAMTEC_MTSW-101-X-X-D-X, F.Cu at (112.5, 78.5)
- D104, D105: value PMEG3010ESBYL -> CTS05S30; footprint 0_Power:DIODFN100X60X30-2N -> Diode_SMD:D_SOD-882
- D107, D108, D201, D202, D203, D204, D205: value ESD9L1P8 -> RCLAMP01811PW.C; footprint Diode_SMD:D_SOD-882 -> 0_Power:DIODFN100X60X55-2N
- R104: value 330 -> 330R
- SW302: value TS-1088-AR02016 -> EVP-AWED4A; footprint 0_Feedback:SW_TS-1088-AR02016 -> 0_Feedback:SW_EVP-AWED4A
- moved D110 11.0 mm to (125.8, 80.8), turned to -145 degrees
- moved TP107 4.53 mm to (108.0, 95.5)
- moved R108 3.75 mm to (119.0, 85.8)
- moved U104 3.66 mm to (117.0, 85.7)
- moved TP109 1.52 mm to (114.8, 88.5)
- moved TP301 1.00 mm to (109.8, 76.5)
- moved SW302 0.94 mm to (107.0, 81.8)
- moved TP108 0.71 mm to (114.0, 92.5)
- moved TP112 0.65 mm to (104.4, 69.0)
- moved D203 0.64 mm to (102.0, 61.0)
- moved D204 0.61 mm to (100.1, 67.2)
- moved R201 0.58 mm to (102.0, 67.2)
- moved D205 0.51 mm to (97.9, 67.2)
- moved D202 0.46 mm to (97.9, 61.0)
- moved D201 0.45 mm to (99.8, 61.0)
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- renumbered 204 to TP204
Connections:
- C110 pad 1: +3V0 -> /1_Power/LDO_OUT
- C112 pad 1: +1V8_Peripherals -> /1_Power/NPM_VOUT2
- L102 pad 1: +1V8_Peripherals -> /1_Power/NPM_VOUT2
- R108 pad 1: /1_Power/NPM_VOUT1 -> /1_Power/Shunt_CM_Header
- TP105 pad 1: +3V0 -> /1_Power/LDO_OUT
- U101 pad 32: +1V8_Peripherals -> /1_Power/NPM_VOUT2
- U102 pad 1: NC -> unconnected-(U102-NC-Pad1)
- U103 pad 1: +3V0 -> /1_Power/LDO_OUT
- U104 pad 2: /1_Power/NPM_VOUT1 -> /1_Power/Shunt_CM_Header
- U104 pad 3: /1_Power/NPM_VOUT1 -> /1_Power/Shunt_CM_Header
Routing:
- net +1V8_Peripherals: track 140.0 -> 119.3 mm, vias 11 -> 9
- net +3V0: track 55.3 -> 36.7 mm, vias 2 -> 0
- net /1_Power/NPM_VOUT2: track 0.00 -> 18.2 mm, vias 0 -> 2
- net /1_Power/LDO_OUT: track 0.00 -> 15.6 mm, vias 0 -> 2
- net GND: track 84.3 -> 77.5 mm, vias 298 -> 296
- net /1_Power/MCU_CURR_MON_COMP: track 39.3 -> 43.0 mm
- net +1V8_MCU: track 70.8 -> 67.8 mm
- net /1_Power/NPM_VOUT1: track 7.67 -> 6.34 mm
- net /2_nRF Module & NAND Flash + IMU + Magnetometer/ACTUATOR_LOCAL_EN: track 18.7 -> 19.4 mm
- net /1_Power/CHG_DOCK_DET_LPCOMP: track 23.6 -> 24.2 mm
- net /2_nRF Module & NAND Flash + IMU + Magnetometer/ACTUATOR_EXTERNAL_EN: track 39.5 -> 40.0 mm
- net /2_nRF Module & NAND Flash + IMU + Magnetometer/SWD_O: track 36.9 -> 37.4 mm
- net /1_Power/CHG_DOCK_UART_TX: track 25.0 -> 25.6 mm
- net /2_nRF Module & NAND Flash + IMU + Magnetometer/SWD_RESET_MCU: track 29.9 -> 29.4 mm
- added copper zone on F.Cu, net /1_Power/NPM_VOUT2
- added copper zone on F.Cu, net /1_Power/Shunt_CM_Header
- removed copper zone on F.Cu, net +1V8_Peripherals

Commit message: created gerbers and drills
Parts:
- moved BT101 2.25 mm to (138.6, 79.5)
- moved J301 2.00 mm to (115.5, 58.0)
- moved M401 2.00 mm to (110.8, 65.0)
- moved MH302 2.00 mm to (92.2, 59.2)
- moved MH303 2.00 mm to (141.2, 59.2)
- moved TP302 2.00 mm to (123.2, 58.0)
- moved TP112 1.63 mm to (105.7, 68.0)
- moved D302 1.05 mm to (117.8, 61.2)
- moved D301 0.75 mm to (110.8, 71.2)
- moved Q301 0.75 mm to (110.8, 72.8)
- moved D203 0.59 mm to (102.2, 60.5)
- moved D201 0.59 mm to (100.0, 60.5)
- moved D110 0.58 mm to (126.2, 80.5)
- moved D202 0.56 mm to (97.9, 60.5)
- moved R201 0.30 mm to (102.3, 67.2)
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Routing:
- net Net-(D302-A): track 5.64 -> 8.72 mm
- net /2_nRF Module & NAND Flash + IMU + Magnetometer/ACTUATOR_EXTERNAL_EN: track 40.0 -> 42.8 mm
- net +3V0: track 36.7 -> 39.5 mm
- net /2_nRF Module & NAND Flash + IMU + Magnetometer/SWD_O: track 37.4 -> 39.9 mm
- net /2_nRF Module & NAND Flash + IMU + Magnetometer/SWD_CLK: track 35.0 -> 37.4 mm
- net /1_Power/BAT-: track 24.6 -> 26.8 mm
- net Net-(D301-A): track 6.46 -> 8.33 mm
- net +VBAT: track 30.4 -> 32.2 mm
- net /2_nRF Module & NAND Flash + IMU + Magnetometer/SWD_IO: track 31.1 -> 32.4 mm
- net GND: track 77.5 -> 76.3 mm, vias 296 -> 302
- net /2_nRF Module & NAND Flash + IMU + Magnetometer/ACTUATOR_LOCAL_EN: track 19.4 -> 20.1 mm
- net +1V8_MCU: track 67.8 -> 68.3 mm
Other:
- board size 55 x 53 mm -> 55 x 55 mm
