File: IEMU_Memory_Eval/IEMU_Memory_Eval.kicad_pcb (KiCad board)
At the start: 4 copper layers, 29.5 x 36.5 mm, 20 parts, among them J1 2211S-02G, J2 2211S-02G, J3 2211S-02G, J4 2211S-02G, J5 2211S-02G, J6 2211S-02G, J7 2211S-02G, J8 2211S-02G, J9 Conn_02x14_Counter_Clockwise, U1 TPS22917DBV, U2 MT29F2G01ABAGDWB-IT:G

Commit message: added the carrier board
Connections:
- J9 pad 14: unconnected-(J9-Pin_14-Pad14) -> GND
- J9 pad 15: unconnected-(J9-Pin_15-Pad15) -> GND
- J9 pad 28: unconnected-(J9-Pin_28-Pad28) -> GND
