File: IEMU_Memory_Eval/IEMU_Memory_Eval.kicad_sch (KiCad schematic)
At the start: 20 parts, among them J1 2211S-02G, J2 2211S-02G, J3 2211S-02G, J4 2211S-02G, J5 2211S-02G, J6 2211S-02G, J7 2211S-02G, J8 2211S-02G, J9 Conn_02x14_Counter_Clockwise, U1 TPS22917DBV, U2 MT29F2G01ABAGDWB-IT:G

Commit message: added the carrier board
Connections:
- net GND: now also J9.14 (Pin_14), J9.15 (Pin_15), J9.28 (Pin_28)
- no-connect marks 21 -> 18
Changed lines of the file:
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@@
+	)
+	(junction
+		(at 257.81 135.89)
+		(diameter 0)
+		(color 0 0 0 0)
+	)
+	(junction
+		(at 223.52 135.89)
+		(diameter 0)
+		(color 0 0 0 0)
 	)
 	(junction
@@
 	)
 	(no_connect
-		(at 251.46 135.89)
-	)
-	(no_connect
-		(at 238.76 135.89)
-	)
-	(no_connect
 		(at 251.46 130.81)
 	)
@@
 	)
 	(no_connect
+		(at 238.76 118.11)
+	)
+	(no_connect
 		(at 251.46 133.35)
 	)
 	(no_connect
+		(at 238.76 123.19)
+	)
+	(no_connect
 		(at 251.46 125.73)
 	)
 	(no_connect
-		(at 251.46 102.87)
-	)
-	(no_connect
 		(at 251.46 123.19)
 	)
@@
 	)
 	(no_connect
-		(at 238.76 123.19)
-	)
-	(no_connect
 		(at 71.12 64.77)
 	)
@@
 	)
 	(no_connect
-		(at 238.76 118.11)
-	)
-	(no_connect
 		(at 251.46 118.11)
 	)
@@
 	(wire
 		(pts
+			(xy 223.52 105.41) (xy 238.76 105.41)
+		)
+		(stroke
+			(width 0)
+			(type default)
+		)
+	)
+	(wire
+		(pts
+			(xy 223.52 137.16) (xy 223.52 135.89)
+		)
+		(stroke
+			(width 0)
+			(type default)
+		)
+	)
+	(wire
+		(pts
 			(xy 204.47 45.72) (xy 204.47 43.18)
 		)
@@
 	(wire
 		(pts
-			(xy 228.6 105.41) (xy 238.76 105.41)
-		)
-		(stroke
-			(width 0)
-			(type default)
-		)
-	)
-	(wire
-		(pts
 			(xy 116.84 128.27) (xy 116.84 127)
 		)
@@
 	(wire
 		(pts
+			(xy 251.46 135.89) (xy 257.81 135.89)
+		)
+		(stroke
+			(width 0)
+			(type default)
+		)
+	)
+	(wire
+		(pts
 			(xy 144.78 62.23) (xy 149.86 62.23)
 		)
@@
 	(wire
 		(pts
+			(xy 257.81 135.89) (xy 257.81 137.16)
+		)
+		(stroke
+			(width 0)
+			(type default)
+		)
+	)
+	(wire
+		(pts
 			(xy 196.85 53.34) (xy 196.85 67.31)
 		)
@@
 	(wire
 		(pts
+			(xy 257.81 102.87) (xy 257.81 135.89)
+		)
+		(stroke
+			(width 0)
+			(type default)
+		)
+	)
+	(wire
+		(pts
+			(xy 223.52 135.89) (xy 238.76 135.89)
+		)
+		(stroke
+			(width 0)
+			(type default)
+		)
+	)
+	(wire
+		(pts
 			(xy 189.23 43.18) (xy 196.85 43.18)
 		)
@@
 		(pts
 			(xy 204.47 64.77) (xy 207.01 64.77)
+		)
+		(stroke
+			(width 0)
+			(type default)
+		)
+	)
+	(wire
+		(pts
+			(xy 223.52 105.41) (xy 223.52 135.89)
+		)
+		(stroke
+			(width 0)
+			(type default)
+		)
+	)
+	(wire
+		(pts
+			(xy 251.46 102.87) (xy 257.81 102.87)
 		)
 		(stroke
@@
 	(symbol
 		(lib_id "power:GND")
-		(at 228.6 105.41 0)
+		(at 257.81 137.16 0)
+		(unit 1)
+		(exclude_from_sim no)
+		(in_bom yes)
+		(on_board yes)
+		(dnp no)
+		(fields_autoplaced yes)
+		(property "Reference" "#PWR0114"
+			(at 257.81 143.51 0)
+			(effects
+				(font
+					(size 1.27 1.27)
+				)
+				(hide yes)
+			)
+		)
+		(property "Value" "GND"
+			(at 257.81 140.97 0)
+			(effects
+				(font
+					(size 1.27 1.27)
+				)
+				(hide yes)
+			)
+		)
+		(property "Footprint" ""
+			(at 257.81 137.16 0)
+			(effects
+				(font
+					(size 1.27 1.27)
+				)
+				(hide yes)
+			)
+		)
+		(property "Datasheet" ""
+			(at 257.81 137.16 0)
+			(effects
+				(font
+					(size 1.27 1.27)
+				)
+				(hide yes)
+			)
+		)
+		(property "Description" "Power symbol creates a global label with name \"GND\" , ground"
+			(at 257.81 137.16 0)
+			(effects
+				(font
+					(size 1.27 1.27)
+				)
+				(hide yes)
+			)
+		)
+		(pin "1"
+		)
+		(instances
+			(project "IEMU_Memory_Eval"
+				(path "/9e49c642-f255-427f-a9b3-c443921843be"
+					(reference "#PWR0114")
+					(unit 1)
+				)
+			)
+		)
+	)
+	(symbol
+		(lib_id "power:GND")
+		(at 223.52 137.16 0)
 		(unit 1)
 		(exclude_from_sim no)
@@
 		(fields_autoplaced yes)
 		(property "Reference" "#PWR0101"
-			(at 228.6 111.76 0)
+			(at 223.52 143.51 0)
 			(effects
 				(font
@@
 		)
 		(property "Value" "GND"
-			(at 228.6 109.22 0)
+			(at 223.52 140.97 0)
 			(effects
 				(font
@@
 		)
 		(property "Footprint" ""
-			(at 228.6 105.41 0)
+			(at 223.52 137.16 0)
 			(effects
 				(font
@@
 		)
 		(property "Datasheet" ""
-			(at 228.6 105.41 0)
+			(at 223.52 137.16 0)
 			(effects
 				(font
@@
 		)
 		(property "Description" "Power symbol creates a global label with name \"GND\" , ground"
-			(at 228.6 105.41 0)
-			(effects
-				(font
+			(at 223.52 137.16 0)
+			(effects
+				(font

Commit message: final changes before order, including a clutch swd connector change
Parts:
- C1: Distributor Link 1 https://de.farnell.com/samsung-electro-mechanics/cl05b104ko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 -> https://de.farnell.com/tdk/c1005x5r1a475k050bc/kondensator-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; Distributor Link 2 https://www.digikey.de/de/products/detail/samsung-electro-m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 -> (none); LCSC C1525 -> (none); Manufacturer_Name Samsung Electro-Mechanics -> TDK; Manufacturer_Part_Number CL05B104KO5NNNC -> C1005X5R1A475K050BC
Changed lines of the file:
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@@
 			)
 		)
-		(property "Datasheet" "https://www.lcsc.com/datasheet/C1525.pdf"
+		(property "Datasheet" "https://www.farnell.com/datasheets/4520405.pdf"
 			(at 104.648 89.154 0)
 			(effects
@@
 			)
 		)
-		(property "Description" "100nF 16V X7R ±10% 0402 Multilayer Ceramic Capacitors MLCC - SMD/SMT ROHS"
+		(property "Description" "Keramikvielschichtkondensator, SMD, 4.7 µF, 10 V, 0402 [Metrisch 1005], ± 10%, X5R"
 			(at 105.41 78.994 0)
 			(effects
@@
 			)
 		)
-		(property "Manufacturer_Name" "Samsung Electro-Mechanics"
+		(property "Manufacturer_Name" "TDK"
 			(at 103.124 83.82 0)
 			(effects
@@
 			)
 		)
-		(property "Manufacturer_Part_Number" "CL05B104KO5NNNC"
+		(property "Manufacturer_Part_Number" "C1005X5R1A475K050BC"
 			(at 104.394 99.314 0)
 			(effects
@@
 			)
 		)
-		(property "Distributor Link 1" "https://de.farnell.com/samsung-electro-mechanics/cl05b104ko5nnnc/kondensator-0-1uf-16v-mlcc-0402/dp/3013349"
-			(at 107.95 92.456 0)
+		(property "Distributor Link 1" "https://de.farnell.com/tdk/c1005x5r1a475k050bc/kondensator-4-7-f-10v-10-x5r-0402/dp/2528756"
+			(at 102.87 66.04 0)
 			(effects
 				(font
-					(size 1.27 1.27)
-				)
-				(hide yes)
-			)
-		)
-		(property "Distributor Link 2" "https://www.digikey.de/de/products/detail/samsung-electro-mechanics/CL05B104KO5NNNC/3886659?s=N4IgTCBcDaIMIBkAMBWAQgRiQFgNIHkUA5EuEAXQF8g"
-			(at 108.458 94.488 0)
-			(effects
-				(font
-					(size 1.27 1.27)
-				)
-				(hide yes)
-			)
-		)
-		(property "LCSC" "C1525"
-			(at 107.442 72.136 0)
-			(effects
-				(font
