File: IEMU_Power_Eval/IEMU_Power_Eval.kicad_pcb (KiCad board)
At the start: 4 copper layers, 36.6 x 45.2 mm, 37 parts, among them J1 USB4125-GF-A, J2 Conn_01x02, J3 Conn_01x02, J4 Conn_02x14_Counter_Clockwise, Q1 CSD85301Q2, SW1 SW_Push, U1 NPM1304-QEAA-R7, U2 BQ29702DSER

Commit message: small changes
Routing:
- net GND: vias 132 -> 134
Other:
- outline, holes or cut-outs redrawn
Changed lines of the file:
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@@
 	)
 	(gr_line
-		(start 41.35 57)
+		(start 41.35 55.5)
 		(end 41.35 92.3)
 		(stroke
@@
 	)
 	(gr_arc
-		(start 41.35 57)
-		(mid 42.082233 55.232233)
-		(end 43.85 54.5)
+		(start 41.35 55.5)
+		(mid 41.642893 54.792893)
+		(end 42.35 54.5)
 		(stroke
 			(width 0.05)
@@
 	(gr_line
 		(start 77.95 92.3)
-		(end 77.95 57)
+		(end 77.95 55.5)
 		(stroke
 			(width 0.05)
@@
 	)
 	(gr_arc
-		(start 75.45 54.5)
-		(mid 77.217767 55.232233)
-		(end 77.95 57)
+		(start 76.95 54.5)
+		(mid 77.657107 54.792893)
+		(end 77.95 55.5)
 		(stroke
 			(width 0.05)
@@
 	)
 	(gr_line
-		(start 75.45 54.5)
-		(end 43.85 54.5)
+		(start 76.95 54.5)
+		(end 42.35 54.5)
 		(stroke
 			(width 0.05)
@@
 	)
 	(via
+		(at 76.15 55.55)
+		(size 0.6)
+		(drill 0.3)
+		(layers "F.Cu" "B.Cu")
+		(free yes)
+		(net 4)
+	)
+	(via
 		(at 45.15 63.3)
 		(size 0.6)
@@
 		(size 0.6)
 		(drill 0.3)
+		(layers "F.Cu" "B.Cu")
+		(free yes)
+		(net 4)
+	)
+	(via
+		(at 43.15 55.55)
+		(size 0.6)
+		(drill 0.3)
