File: IEMU_Carrier_Eval/IEMU_carrier_eval.kicad_pcb (KiCad board)
At the start: 4 copper layers, 106.3 x 93.6 mm, 7 parts, among them J1 Conn_02x14_Socket, J2 Conn_02x14_Socket, J3 Conn_02x14_Socket, J4 Conn_02x12_Socket, J5 Conn_02x14_Socket, J6 Conn_02x12_Socket, J7 Conn_01x12_Socket

Commit message: final changes before order, including a clutch swd connector change
Parts:
- added H1: MountingHole_Pad, MountingHole:MountingHole_1.2mm_M2_Pad_Via, F.Cu at (58.5, 50.6)
- added H2: MountingHole_Pad, MountingHole:MountingHole_1.2mm_M2_Pad_Via, F.Cu at (132.9, 50.6)
- added H3: MountingHole_Pad, MountingHole:MountingHole_1.2mm_M2_Pad_Via, F.Cu at (70.0, 131.3)
- added H4: MountingHole_Pad, MountingHole:MountingHole_1.2mm_M2_Pad_Via, F.Cu at (117.0, 131.3)
