File: IEMU_Carrier_Eval/IEMU_carrier_eval.kicad_sch (KiCad schematic)
At the start: 7 parts, among them J1 Conn_02x14_Socket, J2 Conn_02x14_Socket, J3 Conn_02x14_Socket, J4 Conn_02x12_Socket, J5 Conn_02x14_Socket, J6 Conn_02x12_Socket, J7 Conn_01x12_Socket

Commit message: final changes before order, including a clutch swd connector change
Parts:
- added H1, H2, H3, H4: MountingHole_Pad, MountingHole:MountingHole_1.2mm_M2_Pad_Via, symbol Mechanical:MountingHole_Pad
Connections:
- net GND: now also H1.1, H2.1, H3.1, H4.1
