File: IEMU_Sensor_Core/IEMU_Sensor_Core.kicad_pcb (KiCad board)
At the start: 4 copper layers, 37 x 64.5 mm, 27 parts, among them J1 MTSW-103-07-T-S-240, J2 MTSW-101-07-T-D-240, J3 MTSW-101-07-T-D-240, J4 SSW-105-02-T-D-RA, J5 Conn_02x14_Counter_Clockwise, Q1 INA216A2RSWR, U1 Ezurio BL54L15, Y1 32.768kHz

Commit message: final changes before order, including a clutch swd connector change
Parts:
- J4: footprint 0_Connectors:SSW-105-XX-YYY-D-RA -> 0_Connectors:PinHeader_2x05_P1.27mm_Vertical_SWD_Debug
- moved TP7 5.66 mm to (87.0, 59.3)
- moved J4 4.13 mm to (89.4, 50.5), turned to 0 degrees
- moved TP8 3.06 mm to (82.7, 59.4)
- moved R3 2.00 mm to (82.8, 56.8), turned to 0 degrees
- moved C3 0.15 mm to (80.0, 53.2)
Connections:
- net /ANI_1 renamed /AIN_1
- net /ANI_2 renamed /AIN_2
Routing:
- net /SWD_O: track 9.53 -> 23.9 mm
- net /SWD_CLK: track 7.99 -> 21.3 mm
- net /SWD_IO: track 9.67 -> 18.3 mm
- net GND: track 18.3 -> 12.2 mm, vias 270 -> 289
- net /SWD_RST_CONN: track 6.01 -> 11.3 mm, vias 0 -> 1
- net /+VDD_NRF: track 57.6 -> 62.0 mm, vias 3 -> 4
- net /SWD_RST_MCU: track 6.86 -> 9.08 mm
- net /GPIO_2: track 51.2 -> 49.1 mm, vias 2 -> 4
- net /GPIO_1: track 54.3 -> 55.0 mm
Other:
- board text added: "SWD"
