File: IEMU_Sensor_Core/IEMU_Sensor_Core.kicad_sch (KiCad schematic)
At the start: 27 parts, among them J1 MTSW-103-07-T-S-240, J2 MTSW-101-07-T-D-240, J3 MTSW-101-07-T-D-240, J4 SSW-105-02-T-D-RA, J5 Conn_02x14_Counter_Clockwise, Q1 INA216A2RSWR, U1 Ezurio BL54L15, Y1 32.768kHz

Commit message: added memory board and refined vibration board details
Connections:
- net ANI_1 renamed AIN_1
- net ANI_2 renamed AIN_2
Other:
- company: (none) -> Mustafa Acar
- title: (none) -> IEMU Sensor - Evaluation Board
Changed lines of the file:
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@@
 	(generator_version "9.0")
 	(paper "A4")
+	(title_block
+		(title "IEMU Sensor - Evaluation Board")
+		(date "2026-10-09")
+		(rev "0.1")
+		(company "Mustafa Acar")
+	)
 	(text "As GND reference\nfor the power profiler"
 		(exclude_from_sim no)
@@
 		)
 	)
-	(label "ANI_2"
+	(label "AIN_2"
 		(at 254 100.33 180)
 		(effects
@@
 		)
 	)
-	(label "ANI_1"
+	(label "AIN_1"
 		(at 128.27 66.04 180)
 		(effects
@@
 		)
 	)
-	(label "ANI_1"
+	(label "AIN_1"
 		(at 254 97.79 180)
 		(effects
@@
 		)
 	)
-	(label "ANI_2"
+	(label "AIN_2"
 		(at 128.27 62.23 180)
 		(effects

Commit message: final changes before order, including a clutch swd connector change
Parts:
- J4: footprint 0_Connectors:SSW-105-XX-YYY-D-RA -> 0_Connectors:PinHeader_2x05_P1.27mm_Vertical_SWD_Debug; Distributor Link 1 https://de.farnell.com/samtec/ssw-105-02-t-d-ra/buchse-2-54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 -> https://de.farnell.com/samtec/ftsh-105-01-f-d-k/stiftleiste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; Manufacturer_Part_Number SSW-105-02-T-D-RA -> FTSH-105-01-F-D-K
Changed lines of the file:
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@@
 			)
 		)
-		(property "Footprint" "0_Connectors:SSW-105-XX-YYY-D-RA"
+		(property "Footprint" "0_Connectors:PinHeader_2x05_P1.27mm_Vertical_SWD_Debug"
 			(at 229.87 -39.04 0)
 			(effects
@@
 			)
 		)
-		(property "Datasheet" "https://suddendocs.samtec.com/productspecs/tsw-sxx.pdf"
+		(property "Datasheet" "https://www.farnell.com/datasheets/4639383.pdf"
 			(at 229.87 -139.04 0)
 			(effects
@@
 			)
 		)
-		(property "Description" "10-polige, 2-reihige Buchsenleiste mit 0.635mm-Vierkantstiften mit Mattverzinnung, einem Rastermaß von 2.54mm"
+		(property "Description" "Stiftleiste, Board-to-Board, Wire-to-Board, 1.27 mm, 2 Reihe(n), 10 Kontakt(e), Durchsteckmontage"
 			(at 235.966 66.802 0)
 			(effects
@@
 			)
 		)
-		(property "Manufacturer_Part_Number" "SSW-105-02-T-D-RA"
+		(property "Manufacturer_Part_Number" "FTSH-105-01-F-D-K"
 			(at 229.87 -739.04 0)
 			(effects
@@
 			)
 		)
-		(property "Distributor Link 1" "https://de.farnell.com/samtec/ssw-105-02-t-d-ra/buchse-2-54mm-ra-10pol/dp/2308470?MER=sy-me-pd-mi-alte"
+		(property "Distributor Link 1" "https://de.farnell.com/samtec/ftsh-105-01-f-d-k/stiftleiste-10p-2r-1-27mm-tht/dp/2856426"
 			(at 248.92 55.88 0)
 			(effects
-				(font
-					(size 1.27 1.27)
-				)
-				(hide yes)
-			)
-		)
-		(property "Distributor_Link_1" ""
-			(at 248.92 55.88 0)
-			(effects
