File: IEMU_Vib_Eval/IEMU_Vib_Eval.kicad_pcb (KiCad board)
At the start: 4 copper layers, 37.2 x 26 mm, 10 parts, among them J1 Conn_02x14_Counter_Clockwise, M1 VG0832012, U101 TPS22917DBV, U102 DRV8210DRL

Commit message: added memory board and refined vibration board details
Parts:
- added R1: 510k, Resistor_SMD:R_0603_1608Metric, F.Cu at (189.4, 101.0)
- renumbered R101 to R2
Routing:
- net /VIB_EN: track 14.4 -> 19.6 mm
- net GND: vias 5 -> 45

Commit message: added the carrier board
Connections:
- J1 pad 14: unconnected-(J1-Pin_14-Pad14) -> GND
- J1 pad 15: unconnected-(J1-Pin_15-Pad15) -> GND
- J1 pad 20: unconnected-(J1-Pin_20-Pad20) -> GND
- J1 pad 28: unconnected-(J1-Pin_28-Pad28) -> GND
- J1 pad 4: unconnected-(J1-Pin_4-Pad4) -> GND
- J1 pad 6: unconnected-(J1-Pin_6-Pad6) -> GND
- J1 pad 7: /PWM_IN_1 -> /PWM_IN_2
- J1 pad 8: /PWM_IN_2 -> /PWM_IN_1
- J1 pad 9: unconnected-(J1-Pin_9-Pad9) -> GND
- U102 pad 1: /PWM_IN_1 -> /PWM_IN_2
- U102 pad 2: /PWM_IN_2 -> /PWM_IN_1
Other:
- board text added: "GND"
- board text added: "PWM_IN1"
- board text added: "PWM_IN2"
- board text added: "VIB_EN"
- board text added: "V_IN"

Commit message: final changes before order, including a clutch swd connector change
Changed lines of the file:
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@@
 		)
 	)
-	(gr_text "PWM_IN2"
+	(gr_text "PWM_IN1"
 		(at 198.35 98.95 270)
 		(layer "F.SilkS" knockout)
@@
 		)
 	)
-	(gr_text "PWM_IN1"
+	(gr_text "PWM_IN2"
 		(at 195.85 98.95 270)
 		(layer "F.SilkS" knockout)
