File: IEMU_Vib_Eval/IEMU_Vib_Eval.kicad_sch (KiCad schematic)
At the start: 10 parts, among them J1 Conn_02x14_Counter_Clockwise, M1 VG0832012, U101 TPS22917DBV, U102 DRV8210DRL

Commit message: added memory board and refined vibration board details
Parts:
- added R1: 510k, Resistor_SMD:R_0603_1608Metric, symbol 0_Passives:R_510k
- C5: Distributor Link 1 (none) -> https://de.farnell.com/samsung-electro-mechanics/cl05b104ko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; Manufacturer_Name (none) -> Samsung Electro-Mechanics; Manufacturer_Part_Number (none) -> CL05B104KO5NNNC
- J1: Distributor Link 1 (none) -> https://de.farnell.com/multicomp-pro/mc34735/stecker-1-reih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; Manufacturer_Name (none) -> MULTICOMP PRO; Manufacturer_Part_Number (none) -> MC34735
- R2: renamed from R101; Distributor Link 1 (none) -> https://de.farnell.com/vishay/rca0805100rfkea/dickschichtwi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; Manufacturer_Name (none) -> VISHAY; Manufacturer_Part_Number (none) -> RCA0805100RFKEA
Connections:
- net GND: now also R1.2
- net VIB_EN: now also R1.1
Other:
- note added: "H-bridge; mcu switches it via PWM"
- note added: "LRA vibration motor"
- note added: "caps act as energy buffer for the LRA, as the coin cell can't supply the peak currents"
- note added: "decouples the motor's current peaks from the battery and protects the nRF's supply"
- company: (none) -> Mustafa Acar
- title: (none) -> Vibration-Motor Evaluation-Board

Commit message: added the carrier board
Connections:
- net GND: now also J1.14 (Pin_14), J1.15 (Pin_15), J1.20 (Pin_20), J1.28 (Pin_28), J1.4 (Pin_4), J1.6 (Pin_6), J1.9 (Pin_9)
- net PWM_IN_1: now also J1.8 (Pin_8), U102.2 (IN2); no longer J1.7 (Pin_7), U102.1 (IN1)
- net PWM_IN_2: now also J1.7 (Pin_7), U102.1 (IN1); no longer J1.8 (Pin_8), U102.2 (IN2)
- no-connect marks 25 -> 18
Other:
- moved on the sheet: J1
